Commit message: translate to real DynaArm position

File: urdf/dynaarm_standalone.urdf (robot description, URDF)
Before this commit: robot dynaarm, 12 links, 11 joints
Links:
- removed link table
- added link arm_base_link
- added link base_link
Joints:
- removed joint table_joint
- added joint base_to_arm: type fixed, parent base_link, child arm_base_link, origin xyz=0.3 0 0.595 rpy=0 0 3.141592653589793
- added joint world_to_base: type fixed, parent world, child base_link, origin xyz=0 0 0 rpy=0 0 0
- joint joint_base: parent table -> arm_base_link
